File: Schematic rob/Schematic rob.kicad_pcb (KiCad board)
At the start: 0 parts

Commit message: Updated schematic and added datasheets
Parts:
- added Q1: C2M0080120D, Package_TO_SOT_THT:TO-247-3_Vertical, F.Cu at (125.0, 83.6)
- added Q2: C2M0080120D, Package_TO_SOT_THT:TO-247-3_Vertical, F.Cu at (125.0, 90.2)
Other:
- copper layers 0 -> 2
Changed lines of the file:
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@@
 (kicad_pcb (version 20230517) (generator pcbnew)
+  (general
+    (thickness 1.6)
+  )
+  (paper "A4")
+  (layers
+    (0 "F.Cu" signal)
+    (31 "B.Cu" signal)
+    (32 "B.Adhes" user "B.Adhesive")
+    (33 "F.Adhes" user "F.Adhesive")
+    (34 "B.Paste" user)
+    (35 "F.Paste" user)
+    (36 "B.SilkS" user "B.Silkscreen")
+    (37 "F.SilkS" user "F.Silkscreen")
+    (38 "B.Mask" user)
+    (39 "F.Mask" user)
+    (40 "Dwgs.User" user "User.Drawings")
+    (41 "Cmts.User" user "User.Comments")
+    (42 "Eco1.User" user "User.Eco1")
+    (43 "Eco2.User" user "User.Eco2")
+    (44 "Edge.Cuts" user)
+    (45 "Margin" user)
+    (46 "B.CrtYd" user "B.Courtyard")
+    (47 "F.CrtYd" user "F.Courtyard")
+    (48 "B.Fab" user)
+    (49 "F.Fab" user)
+    (50 "User.1" user)
+    (51 "User.2" user)
+    (52 "User.3" user)
+    (53 "User.4" user)
+    (54 "User.5" user)
+    (55 "User.6" user)
+    (56 "User.7" user)
+    (57 "User.8" user)
+    (58 "User.9" user)
+  )
+  (setup
+    (pad_to_mask_clearance 0)
+    (pcbplotparams
+      (layerselection 0x00010fc_ffffffff)
+      (plot_on_all_layers_selection 0x0000000_00000000)
+      (disableapertmacros false)
+      (usegerberextensions false)
+      (usegerberattributes true)
+      (usegerberadvancedattributes true)
+      (creategerberjobfile true)
+      (dashed_line_dash_ratio 12.000000)
+      (dashed_line_gap_ratio 3.000000)
+      (svgprecision 4)
+      (plotframeref false)
+      (viasonmask false)
+      (mode 1)
+      (useauxorigin false)
+      (hpglpennumber 1)
+      (hpglpenspeed 20)
+      (hpglpendiameter 15.000000)
+      (pdf_front_fp_property_popups true)
+      (pdf_back_fp_property_popups true)
+      (dxfpolygonmode true)
+      (dxfimperialunits true)
+      (dxfusepcbnewfont true)
+      (psnegative false)
+      (psa4output false)
+      (plotreference true)
+      (plotvalue true)
+      (plotinvisibletext false)
+      (sketchpadsonfab false)
+      (subtractmaskfromsilk false)
+      (outputformat 1)
+      (mirror false)
+      (drillshape 1)
+      (scaleselection 1)
+      (outputdirectory "")
+    )
+  )
+  (net 0 "")
+  (net 1 "unconnected-(Q1-G-Pad1)")
+  (net 2 "Net-(D14-K)")
+  (net 3 "Net-(D1-K)")
+  (net 4 "unconnected-(Q2-G-Pad1)")
+  (net 5 "Net-(Q2-S)")
+  (footprint "Package_TO_SOT_THT:TO-247-3_Vertical" (layer "F.Cu")
+    (at 124.99 90.17)
+    (descr "TO-247-3, Vertical, RM 5.45mm, see https://toshiba.semicon-storage.com/us/product/mosfet/to-247-4l.html")
+    (tags "TO-247-3 Vertical RM 5.45mm")
+    (property "Sheetfile" "Schematic rob.kicad_sch")
+    (property "Sheetname" "")
+    (property "ki_description" "36A Id, 1200V Vds, 80mOhm, N-Channel SiC MOSFET, TO-247")
+    (property "ki_keywords" "N-Channel SiC MOSFET")
+    (attr through_hole)
+    (fp_text reference "Q2" (at 5.45 -3.45) (layer "F.SilkS")
+      (effects (font (size 1 1) (thickness 0.15)))
+    )
+    (fp_text value "C2M0080120D" (at 5.45 3.95) (layer "F.Fab")
+      (effects (font (size 1 1) (thickness 0.15)))
+    )
+    (fp_line (start -2.62 -2.451) (end -2.62 2.82)
+      (stroke (width 0.12) (type solid)) (layer "F.SilkS"))
+    (fp_line (start -2.62 -2.451) (end 13.52 -2.451)
+      (stroke (width 0.12) (type solid)) (layer "F.SilkS"))
+    (fp_line (start -2.62 2.82) (end 13.52 2.82)
+      (stroke (width 0.12) (type solid)) (layer "F.SilkS"))
+    (fp_line (start 3.646 -2.451) (end 3.646 2.82)
+      (stroke (width 0.12) (type solid)) (layer "F.SilkS"))
+    (fp_line (start 7.255 -2.451) (end 7.255 2.82)
+      (stroke (width 0.12) (type solid)) (layer "F.SilkS"))
+    (fp_line (start 13.52 -2.451) (end 13.52 2.82)
+      (stroke (width 0.12) (type solid)) (layer "F.SilkS"))
+    (fp_line (start -2.75 -2.59) (end -2.75 2.95)
+      (stroke (width 0.05) (type solid)) (layer "F.CrtYd"))
+    (fp_line (start -2.75 2.95) (end 13.65 2.95)
+      (stroke (width 0.05) (type solid)) (layer "F.CrtYd"))
+    (fp_line (start 13.65 -2.59) (end -2.75 -2.59)
+      (stroke (width 0.05) (type solid)) (layer "F.CrtYd"))
+    (fp_line (start 13.65 2.95) (end 13.65 -2.59)
+      (stroke (width 0.05) (type solid)) (layer "F.CrtYd"))
+    (fp_line (start -2.5 -2.33) (end -2.5 2.7)
+      (stroke (width 0.1) (type solid)) (layer "F.Fab"))
+    (fp_line (start -2.5 2.7) (end 13.4 2.7)
+      (stroke (width 0.1) (type solid)) (layer "F.Fab"))
+    (fp_line (start 3.645 -2.33) (end 3.645 2.7)
+      (stroke (width 0.1) (type solid)) (layer "F.Fab"))
+    (fp_line (start 7.255 -2.33) (end 7.255 2.7)
+      (stroke (width 0.1) (type solid)) (layer "F.Fab"))
+    (fp_line (start 13.4 -2.33) (end -2.5 -2.33)
+      (stroke (width 0.1) (type solid)) (layer "F.Fab"))
+    (fp_line (start 13.4 2.7) (end 13.4 -2.33)
+      (stroke (width 0.1) (type solid)) (layer "F.Fab"))
+    (fp_text user "${REFERENCE}" (at 5.45 -3.45) (layer "F.Fab")
+      (effects (font (size 1 1) (thickness 0.15)))
+    )
+    (pad "1" thru_hole rect (at 0 0) (size 2.5 4.5) (drill 1.5) (layers "*.Cu" "*.Mask")
+      (net 4 "unconnected-(Q2-G-Pad1)") (pinfunction "G") (pintype "input"))
+    (pad "2" thru_hole oval (at 5.45 0) (size 2.5 4.5) (drill 1.5) (layers "*.Cu" "*.Mask")
+      (net 3 "Net-(D1-K)") (pinfunction "D") (pintype "passive"))
+    (pad "3" thru_hole oval (at 10.9 0) (size 2.5 4.5) (drill 1.5) (layers "*.Cu" "*.Mask")
+      (net 5 "Net-(Q2-S)") (pinfunction "S") (pintype "passive"))
+    (model "${KICAD6_3DMODEL_DIR}/Package_TO_SOT_THT.3dshapes/TO-247-3_Vertical.wrl"
+      (offset (xyz 0 0 0))
+      (scale (xyz 1 1 1))
+      (rotate (xyz 0 0 0))
+    )
+  )
+  (footprint "Package_TO_SOT_THT:TO-247-3_Vertical" (layer "F.Cu")
+    (at 124.99 83.58)
+    (descr "TO-247-3, Vertical, RM 5.45mm, see https://toshiba.semicon-storage.com/us/product/mosfet/to-247-4l.html")
+    (tags "TO-247-3 Vertical RM 5.45mm")
+    (property "Note" "Ordered from Amamzon. as FGA25N120 (https://www.amazon.co.jp/-/en/dp/B0BV18ZGTY?psc=1&smid=A2710B5WYUOLWF&ref_=chk_typ_imgToDp)")
+    (property "Sheetfile" "Schematic rob.kicad_sch")
+    (property "Sheetname" "")
+    (property "ki_description" "36A Id, 1200V Vds, 80mOhm, N-Channel SiC MOSFET, TO-247")
+    (property "ki_keywords" "N-Channel SiC MOSFET")
+    (attr through_hole)
+    (fp_text reference "Q1" (at 5.45 -3.45) (layer "F.SilkS")
+      (effects (font (size 1 1) (thickness 0.15)))
+    )
+    (fp_text value "C2M0080120D" (at 5.45 3.95) (layer "F.Fab")
+      (effects (font (size 1 1) (thickness 0.15)))
+    )
+    (fp_line (start -2.62 -2.451) (end -2.62 2.82)
+      (stroke (width 0.12) (type solid)) (layer "F.SilkS"))
+    (fp_line (start -2.62 -2.451) (end 13.52 -2.451)
+      (stroke (width 0.12) (type solid)) (layer "F.SilkS"))
+    (fp_line (start -2.62 2.82) (end 13.52 2.82)
+      (stroke (width 0.12) (type solid)) (layer "F.SilkS"))
+    (fp_line (start 3.646 -2.451) (end 3.646 2.82)
+      (stroke (width 0.12) (type solid)) (layer "F.SilkS"))
+    (fp_line (start 7.255 -2.451) (end 7.255 2.82)
+      (stroke (width 0.12) (type solid)) (layer "F.SilkS"))
+    (fp_line (start 13.52 -2.451) (end 13.52 2.82)
+      (stroke (width 0.12) (type solid)) (layer "F.SilkS"))
+    (fp_line (start -2.75 -2.59) (end -2.75 2.95)
+      (stroke (width 0.05) (type solid)) (layer "F.CrtYd"))
+    (fp_line (start -2.75 2.95) (end 13.65 2.95)
+      (stroke (width 0.05) (type solid)) (layer "F.CrtYd"))
+    (fp_line (start 13.65 -2.59) (end -2.75 -2.59)
+      (stroke (width 0.05) (type solid)) (layer "F.CrtYd"))
+    (fp_line (start 13.65 2.95) (end 13.65 -2.59)
+      (stroke (width 0.05) (type solid)) (layer "F.CrtYd"))
+    (fp_line (start -2.5 -2.33) (end -2.5 2.7)
+      (stroke (width 0.1) (type solid)) (layer "F.Fab"))
+    (fp_line (start -2.5 2.7) (end 13.4 2.7)
+      (stroke (width 0.1) (type solid)) (layer "F.Fab"))
+    (fp_line (start 3.645 -2.33) (end 3.645 2.7)
+      (stroke (width 0.1) (type solid)) (layer "F.Fab"))
+    (fp_line (start 7.255 -2.33) (end 7.255 2.7)
+      (stroke (width 0.1) (type solid)) (layer "F.Fab"))
+    (fp_line (start 13.4 -2.33) (end -2.5 -2.33)
+      (stroke (width 0.1) (type solid)) (layer "F.Fab"))
+    (fp_line (start 13.4 2.7) (end 13.4 -2.33)
+      (stroke (width 0.1) (type solid)) (layer "F.Fab"))
+    (fp_text user "${REFERENCE}" (at 5.45 -3.45) (layer "F.Fab")
+      (effects (font (size 1 1) (thickness 0.15)))
+    )
+    (pad "1" thru_hole rect (at 0 0) (size 2.5 4.5) (drill 1.5) (layers "*.Cu" "*.Mask")
+      (net 1 "unconnected-(Q1-G-Pad1)") (pinfunction "G") (pintype "input"))
+    (pad "2" thru_hole oval (at 5.45 0) (size 2.5 4.5) (drill 1.5) (layers "*.Cu" "*.Mask")
+      (net 2 "Net-(D14-K)") (pinfunction "D") (pintype "passive"))
+    (pad "3" thru_hole oval (at 10.9 0) (size 2.5 4.5) (drill 1.5) (layers "*.Cu" "*.Mask")
+      (net 3 "Net-(D1-K)") (pinfunction "S") (pintype "passive"))
+    (model "${KICAD6_3DMODEL_DIR}/Package_TO_SOT_THT.3dshapes/TO-247-3_Vertical.wrl"
+      (offset (xyz 0 0 0))
+      (scale (xyz 1 1 1))
+      (rotate (xyz 0 0 0))
+    )
+  )
 )

Commit message: updated board data
Parts:
- added U1: Si5351A-B-GT, Package_SO:MSOP-10_3x3mm_P0.5mm, F.Cu at (110.5, 115.6)
- added U3: IR2213, Package_DIP:DIP-14_W7.62mm, F.Cu at (86.4, 100.3)
- added U4: SSD1306, Package_TO_SOT_SMD:SOT-23-5, F.Cu at (113.5, 121.5)
- added U5: ESP32_NODEMCU, Footprints:MODULE_ESP32_NODEMCU, F.Cu at (63.8, 121.9)
- Q1, Q2: value C2M0080120D -> C2M0160120D or C2M0080120D
Connections:
- Q1 pad 1: unconnected-(Q1-G-Pad1) -> Net-(Q1-G)
- Q2 pad 1: unconnected-(Q2-G-Pad1) -> Net-(Q2-G)
